File: KiCAD/Addressable_Coolant_Controller/Addressable_Coolant_Controller.kicad_pcb (KiCad board)
At the start: 2 copper layers, 117.2 x 159.5 mm, 56 parts, among them J1 XW4M-10D2-H1DS, J2 XW4M-02D1-H1DA, K1 G5V-1, K2 G5V-1, K3 G5V-1, K4 G5V-1, K5 G5V-1, K6 G5V-1, K7 G5V-1, K8 G5V-1, U1 ProS3, U10 PC12311NSZ1B, U2 PC12311NSZ1B, U3 PC12311NSZ1B, U4 PC12311NSZ1B, U5 PC12311NSZ1B, U6 PC12311NSZ1B, U7 PC12311NSZ1B, U8 PC12311NSZ1B, U9 PC12311NSZ1B

Commit message: Added second board outline and circular connectors
Parts:
- added J10: 852-002-213R001, 852-002-213R001:852-002-213R001, F.Cu at (301.4, 76.4)
- added J11: 852-002-213R001, 852-002-213R001:852-002-213R001, F.Cu at (313.0, 76.4)
- added J12: 852-004-213R004, 852-002-213R004:852004213R004, F.Cu at (266.7, 190.0)
- added J3: XW4M-12D2-H1DA, xw4m-12d2-h1da:xw4m-12d2-h1da, B.Cu at (275.5, 201.0)
- added J4: 852-002-213R001, 852-002-213R001:852-002-213R001, F.Cu at (301.4, 52.8)
- added J5: 852-002-213R001, 852-002-213R001:852-002-213R001, F.Cu at (313.0, 52.8)
- added J6: 852-002-213R001, 852-002-213R001:852-002-213R001, F.Cu at (324.6, 52.8)
- added J7: 852-002-213R001, 852-002-213R001:852-002-213R001, F.Cu at (301.4, 64.6)
- added J8: 852-002-213R001, 852-002-213R001:852-002-213R001, F.Cu at (313.0, 64.6)
- added J9: 852-002-213R001, 852-002-213R001:852-002-213R001, F.Cu at (324.6, 64.6)
- J1: value XW4M-10D2-H1DS -> XW4M-12D2-H1DA; footprint xw4m-10d2-h1ds:xw4m-10d2-h1ds -> xw4m-12d2-h1da:xw4m-12d2-h1da
- LED5: value C503B-BCN -> C503B-GCN; footprint CreeLED Blue:C503B_BCN_CV0Z0461 -> CreeLED Green:C503B_GCN_CY0C0792
- LED9: value C503B-GCN -> C503B-BCN; footprint CreeLED Green:C503B_GCN_CY0C0792 -> CreeLED Blue:C503B_BCN_CV0Z0461
- R1, R11, R13, R15, R3, R5, R7: value 210Ω -> 1.1kΩ
- R10: value 1.1kΩ -> 2.28kΩ
- R12, R14, R16, R2, R4, R6, R8: value 1.1kΩ -> 210Ω
- R17: value 1.04kΩ -> 1.1kΩ
- R18: value 2.28kΩ -> 210Ω
- R9: value 210Ω -> 1.04kΩ
- U1: value ProS3 -> PC12311NSZ1B; footprint ProS3:ProS3_TH -> PC12311NSZ1B:PC12311NSZ1B
- U10: value PC12311NSZ1B -> ProS3; footprint PC12311NSZ1B:PC12311NSZ1B -> ProS3:ProS3_TH
- moved U9 145.1 mm to (166.1, 178.8)
- moved U1 103.8 mm to (80.8, 57.0)
- moved U2 55.8 mm to (95.0, 57.0)
- moved U3 55.8 mm to (109.2, 57.0)
- moved U4 55.8 mm to (123.4, 57.0)
- moved U5 55.8 mm to (137.6, 57.0)
- moved U6 55.8 mm to (151.8, 57.0)
- moved U7 55.8 mm to (166.0, 57.0)
- moved U8 55.8 mm to (180.2, 57.0)
- moved LED7 43.1 mm to (165.4, 95.4)
- moved LED8 43.1 mm to (179.6, 95.4)
- moved G*** 43.1 mm to (133.2, 155.2)
- moved R17 43.1 mm to (182.4, 169.7)
- moved D1 43.1 mm to (84.7, 84.3)
- moved D3 43.1 mm to (113.0, 84.3)
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Connections:
- J1 pad 1: /S1 -> /Main_Board/S1
- J1 pad 10: GND -> /Main_Board/S8
- J1 pad 11: (no net) -> GND
- J1 pad 12: (no net) -> /Main_Board/MCU GND
- J1 pad 2: /S3 -> /Main_Board/S3
- J1 pad 3: /S5 -> /Main_Board/S5
- J1 pad 4: /S7 -> /Main_Board/S7
- J1 pad 5: GND -> /Main_Board/MCU 3.3v
- J1 pad 6: /S2 -> /Main_Board/IO13
- J1 pad 7: /S4 -> /Main_Board/S2
- J1 pad 8: /S6 -> /Main_Board/S4
- J1 pad 9: /S8 -> /Main_Board/S6
- K1 pad 5: /S1 -> /Main_Board/S8
- K1 pad 6: /S1 -> /Main_Board/S8
- K2 pad 5: /S2 -> /Main_Board/S6
- K2 pad 6: /S2 -> /Main_Board/S6
- K3 pad 5: /S3 -> /Main_Board/S4
- K3 pad 6: /S3 -> /Main_Board/S4
- K4 pad 5: /S4 -> /Main_Board/S3
- K4 pad 6: /S4 -> /Main_Board/S3
- K5 pad 5: /S5 -> /Main_Board/S2
- K5 pad 6: /S5 -> /Main_Board/S2
- K6 pad 5: /S6 -> /Main_Board/S1
- K6 pad 6: /S6 -> /Main_Board/S1
- K7 pad 5: /S7 -> /Main_Board/S5
- K7 pad 6: /S7 -> /Main_Board/S5
- K8 pad 5: /S8 -> /Main_Board/S7
- K8 pad 6: /S8 -> /Main_Board/S7
- R1 pad 1: /MCU 3.3v -> Net-(LED1-Pad1)
- R1 pad 2: Net-(R1-Pad2) -> Net-(D1-A)
- R10 pad 1: Net-(LED5-Pad1) -> Net-(R10-Pad1)
- R10 pad 2: Net-(D5-A) -> GND
- R11 pad 1: /MCU 3.3v -> Net-(LED6-Pad1)
- R11 pad 2: Net-(R11-Pad2) -> Net-(D5-A)
- R12 pad 1: Net-(LED6-Pad1) -> /Main_Board/MCU 3.3v
- R12 pad 2: Net-(D6-A) -> Net-(R12-Pad2)
- R13 pad 1: /MCU 3.3v -> Net-(LED7-Pad1)
- R13 pad 2: Net-(R13-Pad2) -> Net-(D6-A)
- R14 pad 1: Net-(LED7-Pad1) -> /Main_Board/MCU 3.3v
- R14 pad 2: Net-(D7-A) -> Net-(R14-Pad2)
- R15 pad 1: /MCU 3.3v -> Net-(LED8-Pad1)
- R15 pad 2: Net-(R15-Pad2) -> Net-(D7-A)
- R16 pad 1: Net-(LED8-Pad1) -> /Main_Board/MCU 3.3v
- R16 pad 2: Net-(D8-A) -> Net-(R16-Pad2)
- R17 pad 2: GND -> Net-(D8-A)
- R18 pad 1: Net-(R18-Pad1) -> /Main_Board/MCU 3.3v
- R18 pad 2: GND -> Net-(R18-Pad2)
- R2 pad 1: Net-(LED1-Pad1) -> /Main_Board/MCU 3.3v
- R2 pad 2: Net-(D1-A) -> Net-(R2-Pad2)
- R3 pad 1: /MCU 3.3v -> Net-(LED2-Pad1)
- R3 pad 2: Net-(R3-Pad2) -> Net-(D2-A)
- R4 pad 1: Net-(LED2-Pad1) -> /Main_Board/MCU 3.3v
- R4 pad 2: Net-(D2-A) -> Net-(R4-Pad2)
- R5 pad 1: /MCU 3.3v -> Net-(LED3-Pad1)
- R5 pad 2: Net-(R5-Pad2) -> Net-(D3-A)
- R6 pad 1: Net-(LED3-Pad1) -> /Main_Board/MCU 3.3v
- R6 pad 2: Net-(D3-A) -> Net-(R6-Pad2)
- R7 pad 1: /MCU 3.3v -> Net-(LED4-Pad1)
- R7 pad 2: Net-(R7-Pad2) -> Net-(D4-A)
- R8 pad 1: Net-(LED4-Pad1) -> /Main_Board/MCU 3.3v
- R8 pad 2: Net-(D4-A) -> Net-(R8-Pad2)
- R9 pad 1: /MCU 3.3v -> Net-(LED5-Pad1)
- R9 pad 2: Net-(R9-Pad2) -> GND
- U1 pad 1: unconnected-(U1-VBAT-Pad1) -> Net-(R14-Pad2)
- U1 pad 2: unconnected-(U1-GND-Pad2) -> /Main_Board/IO16
- U1 pad 3: unconnected-(U1-5V-Pad3) -> GND
- U1 pad 4: /MCU 3.3v -> Net-(D6-A)
- U10 pad 1: +24V -> unconnected-(U10-VBAT-Pad1)
- U10 pad 2: Net-(R18-Pad1) -> /Main_Board/MCU GND
- U10 pad 3: /IO12 -> unconnected-(U10-5V-Pad3)
- U10 pad 4: /MCU 3.3v -> /Main_Board/MCU 3.3v
- U2 pad 1: Net-(R1-Pad2) -> Net-(R12-Pad2)
- U2 pad 2: /IO16 -> /Main_Board/IO0
- U2 pad 4: Net-(D1-A) -> Net-(D5-A)
- U3 pad 1: Net-(R3-Pad2) -> Net-(R8-Pad2)
- U3 pad 2: /IO0 -> /Main_Board/IO21
- U3 pad 4: Net-(D2-A) -> Net-(D4-A)
- U4 pad 1: Net-(R5-Pad2) -> Net-(R6-Pad2)
- U4 pad 2: /IO21 -> /Main_Board/IO5
- U5 pad 1: Net-(R7-Pad2) -> Net-(R16-Pad2)
- U5 pad 2: /IO5 -> /Main_Board/IO4
- U5 pad 4: Net-(D4-A) -> Net-(D7-A)
- U6 pad 1: Net-(R9-Pad2) -> Net-(R4-Pad2)
- U6 pad 2: /IO4 -> /Main_Board/IO3
- U6 pad 4: Net-(D5-A) -> Net-(D2-A)
- U7 pad 1: Net-(R11-Pad2) -> Net-(R18-Pad2)
- U7 pad 2: /IO3 -> /Main_Board/IO2
- U7 pad 4: Net-(D6-A) -> Net-(D8-A)
- U8 pad 1: Net-(R13-Pad2) -> Net-(R2-Pad2)
- U8 pad 2: /IO2 -> /Main_Board/IO1
- U8 pad 4: Net-(D7-A) -> Net-(D1-A)
- U9 pad 1: Net-(R15-Pad2) -> +24V
- U9 pad 2: /IO1 -> Net-(R10-Pad1)
- U9 pad 3: GND -> /Main_Board/IO12
- U9 pad 4: Net-(D8-A) -> /Main_Board/MCU 3.3v
Routing:
- net (no net): track 0.00 -> 1041.2 mm
- net /MCU 3.3v: track 324.7 -> 0.00 mm
- net /IO1: track 208.9 -> 0.00 mm
- net /Main_Board/IO1: track 0.00 -> 208.9 mm
- net /IO2: track 192.3 -> 0.00 mm
- net /Main_Board/IO2: track 0.00 -> 192.3 mm
- net /Main_Board/IO3: track 0.00 -> 176.6 mm
- net /IO3: track 176.6 -> 0.00 mm
- net /IO4: track 160.9 -> 0.00 mm
- net /Main_Board/IO4: track 0.00 -> 160.9 mm
- net /Main_Board/IO5: track 0.00 -> 144.9 mm
- net /IO5: track 144.9 -> 0.00 mm
- net /Main_Board/IO21: track 0.00 -> 133.3 mm
- net /IO21: track 133.3 -> 0.00 mm
- net /Main_Board/IO0: track 0.00 -> 124.7 mm
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Other:
- board size 117.2 x 159.5 mm -> 210 x 176.5 mm
