File: KiCAD/Addressable_Coolant_Controller/Circular_Connector_Circuit.kicad_sch (KiCad schematic)
At the start: 3 parts, among them J1 852-002-213R001

Commit message: Updating Cree LED footprints with STEP files
Parts:
- LED10: footprint CreeLED Blue:C503B_BCN_CV0Z0461 -> C503B_BCN_CV0Z0461:C503B_BCN_CV0Z0461
Changed lines of the file:
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@@
     (effects (font (size 1.27 1.27)) (justify right))
+  )
+  (netclass_flag "" (length 1) (shape round) (at 132.08 97.79 270) (fields_autoplaced)
+    (effects (font (size 1.27 1.27)) (justify right bottom))
+    (property "Netclass" "power" (at 133.08 97.0915 90)
+      (effects (font (size 1.27 1.27) italic) (justify left) hide)
+    )
   )
   (symbol (lib_id "852-002-213R001:852-002-213R001") (at 106.68 87.63 90) (mirror x) (unit 1)
@@
       (effects (font (size 1.524 1.524)) (justify right))
     )
-    (property "Footprint" "CreeLED Blue:C503B_BCN_CV0Z0461" (at 132.08 85.09 0)
+    (property "Footprint" "C503B_BCN_CV0Z0461:C503B_BCN_CV0Z0461" (at 132.08 85.09 0)
       (effects (font (size 1.27 1.27) italic) hide)
     )
