File: KiCAD/Addressable_Coolant_Controller/Relay_Circuit.kicad_sch (KiCad schematic)
At the start: 6 parts, among them K1 G5V-1, U2 PC12311NSZ1B

Commit message: Updating KiCAD project to multi-board structure
Changed lines of the file:
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@@
     (stroke (width 0) (type default))
+  )
+  (hierarchical_label "GND" (shape input) (at 167.64 111.76 270) (fields_autoplaced)
+    (effects (font (size 1.27 1.27)) (justify right))
   )
   (hierarchical_label "MCU 3.3v" (shape input) (at 118.11 92.71 180) (fields_autoplaced)
     (effects (font (size 1.27 1.27)) (justify right))
+  )
+  (hierarchical_label "+24V" (shape input) (at 152.4 60.96 90) (fields_autoplaced)
+    (effects (font (size 1.27 1.27)) (justify left))
   )
   (hierarchical_label "MCU GPIO" (shape input) (at 125.73 107.95 180) (fields_autoplaced)
@@
     (pin "5")
     (instances
-      (project "Addressable Coolant Controller"
+      (project "Addressable_Coolant_Controller"
         (path "/603d0a2e-fca7-40af-8fa8-51b59d823d4d/9e308de8-a8a3-4754-85bb-a6ac18661119/e62a760e-c259-4531-98bc-86b90a2bedbf"
           (reference "K1") (unit 1)
@@
     (pin "1")
     (instances
-      (project "Addressable Coolant Controller"
+      (project "Addressable_Coolant_Controller"
         (path "/603d0a2e-fca7-40af-8fa8-51b59d823d4d/9e308de8-a8a3-4754-85bb-a6ac18661119/e62a760e-c259-4531-98bc-86b90a2bedbf"
           (reference "R2") (unit 1)
@@
     (pin "4")
     (instances
-      (project "Addressable Coolant Controller"
+      (project "Addressable_Coolant_Controller"
         (path "/603d0a2e-fca7-40af-8fa8-51b59d823d4d/9e308de8-a8a3-4754-85bb-a6ac18661119/e62a760e-c259-4531-98bc-86b90a2bedbf"
           (reference "U2") (unit 1)
@@
     (pin "1")
     (instances
-      (project "Addressable Coolant Controller"
+      (project "Addressable_Coolant_Controller"
         (path "/603d0a2e-fca7-40af-8fa8-51b59d823d4d/9e308de8-a8a3-4754-85bb-a6ac18661119/e62a760e-c259-4531-98bc-86b90a2bedbf"
           (reference "R1") (unit 1)
@@
     (pin "1")
     (instances
-      (project "Addressable Coolant Controller"
+      (project "Addressable_Coolant_Controller"
         (path "/603d0a2e-fca7-40af-8fa8-51b59d823d4d/9e308de8-a8a3-4754-85bb-a6ac18661119/e62a760e-c259-4531-98bc-86b90a2bedbf"
           (reference "LED1") (unit 1)
@@
     (pin "1")
     (instances
-      (project "Addressable Coolant Controller"
-        (path "/603d0a2e-fca7-40af-8fa8-51b59d823d4d/9e308de8-a8a3-4754-85bb-a6ac18661119/e62a760e-c259-4531-98bc-86b90a2bedbf"
-          (reference "D1") (unit 1)
-        )
-        (path "/603d0a2e-fca7-40af-8fa8-51b59d823d4d/9e308de8-a8a3-4754-85bb-a6ac18661119/67f15ca6-662b-4b8a-b540-a2e48d49f414"
-          (reference "D1") (unit 1)
-        )
-        (path "/603d0a2e-fca7-40af-8fa8-51b59d823d4d/9e308de8-a8a3-4754-85bb-a6ac18661119/ed455ca9-960e-4436-b117-323138e12946"
-          (reference "D1") (unit 1)
-        )
-        (path "/603d0a2e-fca7-40af-8fa8-51b59d823d4d/9e308de8-a8a3-4754-85bb-a6ac18661119/30b02bb2-f8cb-4680-8b4d-b295fc1d5eb5"
-          (reference "D1") (unit 1)
-        )
-        (path "/603d0a2e-fca7-40af-8fa8-51b59d823d4d/9e308de8-a8a3-4754-85bb-a6ac18661119/94e5bb90-2559-4272-9ede-e05d2b13ade3"
-          (reference "D1") (unit 1)
-        )
-        (path "/603d0a2e-fca7-40af-8fa8-51b59d823d4d/9e308de8-a8a3-4754-85bb-a6ac18661119/94790e5e-8f24-4c34-8306-22332d8b1ca9"
-          (reference "D1") (unit 1)
-        )
-        (path "/603d0a2e-fca7-40af-8fa8-51b59d823d4d/9e308de8-a8a3-4754-85bb-a6ac18661119/74392b1e-46e8-4b44-bc27-ba912a8cb60e"
-          (reference "D1") (unit 1)
-        )
-        (path "/603d0a2e-fca7-40af-8fa8-51b59d823d4d/9e308de8-a8a3-4754-85bb-a6ac18661119/a5b6bf10-8ef8-4d7b-b15a-e29c9cdfd37d"
-          (reference "D1") (unit 1)
-        )
-      )
-    )
-  )
-  (symbol (lib_id "power:GND") (at 167.64 111.76 0) (unit 1)
-    (in_bom yes) (on_board yes) (dnp no) (fields_autoplaced)
-    (property "Reference" "#PWR04" (at 167.64 118.11 0)
-      (effects (font (size 1.27 1.27)) hide)
-    )
-    (property "Value" "GND" (at 167.64 116.84 0)
-      (effects (font (size 1.27 1.27)))
-    )
-    (property "Footprint" "" (at 167.64 111.76 0)
-      (effects (font (size 1.27 1.27)) hide)
-    )
-    (property "Datasheet" "" (at 167.64 111.76 0)
-      (effects (font (size 1.27 1.27)) hide)
-    )
-    (pin "1")
-    (instances
-      (project "Addressable Coolant Controller"
-        (path "/603d0a2e-fca7-40af-8fa8-51b59d823d4d/9e308de8-a8a3-4754-85bb-a6ac18661119/e62a760e-c259-4531-98bc-86b90a2bedbf"
-          (reference "#PWR04") (unit 1)
-        )
-        (path "/603d0a2e-fca7-40af-8fa8-51b59d823d4d/9e308de8-a8a3-4754-85bb-a6ac18661119/67f15ca6-662b-4b8a-b540-a2e48d49f414"
-          (reference "#PWR04") (unit 1)
-        )
-        (path "/603d0a2e-fca7-40af-8fa8-51b59d823d4d/9e308de8-a8a3-4754-85bb-a6ac18661119/ed455ca9-960e-4436-b117-323138e12946"
-          (reference "#PWR04") (unit 1)
-        )
-        (path "/603d0a2e-fca7-40af-8fa8-51b59d823d4d/9e308de8-a8a3-4754-85bb-a6ac18661119/30b02bb2-f8cb-4680-8b4d-b295fc1d5eb5"
-          (reference "#PWR04") (unit 1)
-        )
-        (path "/603d0a2e-fca7-40af-8fa8-51b59d823d4d/9e308de8-a8a3-4754-85bb-a6ac18661119/94e5bb90-2559-4272-9ede-e05d2b13ade3"
-          (reference "#PWR04") (unit 1)
-        )
-        (path "/603d0a2e-fca7-40af-8fa8-51b59d823d4d/9e308de8-a8a3-4754-85bb-a6ac18661119/94790e5e-8f24-4c34-8306-22332d8b1ca9"
-          (reference "#PWR04") (unit 1)
-        )
-        (path "/603d0a2e-fca7-40af-8fa8-51b59d823d4d/9e308de8-a8a3-4754-85bb-a6ac18661119/74392b1e-46e8-4b44-bc27-ba912a8cb60e"
-          (reference "#PWR04") (unit 1)
-        )
-        (path "/603d0a2e-fca7-40af-8fa8-51b59d823d4d/9e308de8-a8a3-4754-85bb-a6ac18661119/a5b6bf10-8ef8-4d7b-b15a-e29c9cdfd37d"
-          (reference "#PWR04") (unit 1)
-        )
-      )
-    )
-  )
-  (symbol (lib_id "power:+24V") (at 152.4 60.96 0) (unit 1)
-    (in_bom yes) (on_board yes) (dnp no) (fields_autoplaced)
-    (property "Reference" "#PWR03" (at 152.4 64.77 0)
-      (effects (font (size 1.27 1.27)) hide)
-    )
-    (property "Value" "+24V" (at 152.4 55.88 0)
-      (effects (font (size 1.27 1.27)))
-    )
-    (property "Footprint" "" (at 152.4 60.96 0)
-      (effects (font (size 1.27 1.27)) hide)
-    )
-    (property "Datasheet" "" (at 152.4 60.96 0)
-      (effects (font (size 1.27 1.27)) hide)
-    )
-    (pin "1")
-    (instances
-      (project "Addressable Coolant Controller"
-        (path "/603d0a2e-fca7-40af-8fa8-51b59d823d4d/9e308de8-a8a3-4754-85bb-a6ac18661119/e62a760e-c259-4531-98bc-86b90a2bedbf"
-          (reference "#PWR03") (unit 1)
-        )
-        (path "/603d0a2e-fca7-40af-8fa8-51b59d823d4d/9e308de8-a8a3-4754-85bb-a6ac18661119/67f15ca6-662b-4b8a-b540-a2e48d49f414"
-          (reference "#PWR03") (unit 1)
-        )
-        (path "/603d0a2e-fca7-40af-8fa8-51b59d823d4d/9e308de8-a8a3-4754-85bb-a6ac18661119/ed455ca9-960e-4436-b117-323138e12946"
-          (reference "#PWR03") (unit 1)
-        )
-        (path "/603d0a2e-fca7-40af-8fa8-51b59d823d4d/9e308de8-a8a3-4754-85bb-a6ac18661119/30b02bb2-f8cb-4680-8b4d-b295fc1d5eb5"
-          (reference "#PWR03") (unit 1)
-        )
-        (path "/603d0a2e-fca7-40af-8fa8-51b59d823d4d/9e308de8-a8a3-4754-85bb-a6ac18661119/94e5bb90-2559-4272-9ede-e05d2b13ade3"
-          (reference "#PWR03") (unit 1)
-        )
-        (path "/603d0a2e-fca7-40af-8fa8-51b59d823d4d/9e308de8-a8a3-4754-85bb-a6ac18661119/94790e5e-8f24-4c34-8306-22332d8b1ca9"
-          (reference "#PWR03") (unit 1)
-        )
-        (path "/603d0a2e-fca7-40af-8fa8-51b59d823d4d/9e308de8-a8a3-4754-85bb-a6ac18661119/74392b1e-46e8-4b44-bc27-ba912a8cb60e"
-          (reference "#PWR03") (unit 1)
-        )
-        (path "/603d0a2e-fca7-40af-8fa8-51b59d823d4d/9e308de8-a8a3-4754-85bb-a6ac18661119/a5b6bf10-8ef8-4d7b-b15a-e29c9cdfd37d"
-          (reference "#PWR03") (unit 1)
-        )
-      )
+      (project "Addressable_Coolant_Controller"
+        (path "/603d0a2e-fca7-40af-8fa8-51b59d823d4d/9e308de8-a8a3-4754-85bb-a6ac18661119/e62a760e-c259-4531-98bc-86b90a2bedbf"
+          (reference "D1") (unit 1)
+        )
+        (path "/603d0a2e-fca7-40af-8fa8-51b59d823d4d/9e308de8-a8a3-4754-85bb-a6ac18661119/67f15ca6-662b-4b8a-b540-a2e48d49f414"
+          (reference "D1") (unit 1)
+        )
+        (path "/603d0a2e-fca7-40af-8fa8-51b59d823d4d/9e308de8-a8a3-4754-85bb-a6ac18661119/ed455ca9-960e-4436-b117-323138e12946"
+          (reference "D1") (unit 1)
+        )
+        (path "/603d0a2e-fca7-40af-8fa8-51b59d823d4d/9e308de8-a8a3-4754-85bb-a6ac18661119/30b02bb2-f8cb-4680-8b4d-b295fc1d5eb5"
+          (reference "D1") (unit 1)
+        )
+        (path "/603d0a2e-fca7-40af-8fa8-51b59d823d4d/9e308de8-a8a3-4754-85bb-a6ac18661119/94e5bb90-2559-4272-9ede-e05d2b13ade3"
+          (reference "D1") (unit 1)
+        )
+        (path "/603d0a2e-fca7-40af-8fa8-51b59d823d4d/9e308de8-a8a3-4754-85bb-a6ac18661119/94790e5e-8f24-4c34-8306-22332d8b1ca9"
+          (reference "D1") (unit 1)
+        )
+        (path "/603d0a2e-fca7-40af-8fa8-51b59d823d4d/9e308de8-a8a3-4754-85bb-a6ac18661119/74392b1e-46e8-4b44-bc27-ba912a8cb60e"
+          (reference "D1") (unit 1)
+        )
+        (path "/603d0a2e-fca7-40af-8fa8-51b59d823d4d/9e308de8-a8a3-4754-85bb-a6ac18661119/a5b6bf10-8ef8-4d7b-b15a-e29c9cdfd37d"
+          (reference "D1") (unit 1)
+        )
+      )

Commit message: Added voltage divider and changed to 12 pin connectors
Parts:
- renumbered U2 to U1

Commit message: Fixed broken netclasses, removed voltage divider circuit
Other:
- company: (none) -> Warner Consulting Inc.
Changed lines of the file:
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@@
 (kicad_sch (version 20230121) (generator eeschema)
   (paper "A4")
+  (title_block
+    (company "Warner Consulting Inc.")
+  )
   (junction (at 162.56 63.5) (diameter 0) (color 0 0 0 0)
   )

Commit message: Added second board outline and circular connectors
Parts:
- renumbered R2 to R1, R1 to R2, U1 to U8
Changed lines of the file:
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@@
   (symbol (lib_id "Device:R") (at 162.56 82.55 0) (unit 1)
     (in_bom yes) (on_board yes) (dnp no) (fields_autoplaced)
-    (property "Reference" "R2" (at 165.1 81.28 0)
+    (property "Reference" "R1" (at 165.1 81.28 0)
       (effects (font (size 1.27 1.27)) (justify left))
     )
@@
       (project "Addressable_Coolant_Controller"
         (path "/603d0a2e-fca7-40af-8fa8-51b59d823d4d/9e308de8-a8a3-4754-85bb-a6ac18661119/e62a760e-c259-4531-98bc-86b90a2bedbf"
-          (reference "R2") (unit 1)
+          (reference "R1") (unit 1)
         )
         (path "/603d0a2e-fca7-40af-8fa8-51b59d823d4d/9e308de8-a8a3-4754-85bb-a6ac18661119/67f15ca6-662b-4b8a-b540-a2e48d49f414"
-          (reference "R4") (unit 1)
+          (reference "R3") (unit 1)
         )
         (path "/603d0a2e-fca7-40af-8fa8-51b59d823d4d/9e308de8-a8a3-4754-85bb-a6ac18661119/ed455ca9-960e-4436-b117-323138e12946"
-          (reference "R6") (unit 1)
+          (reference "R5") (unit 1)
         )
         (path "/603d0a2e-fca7-40af-8fa8-51b59d823d4d/9e308de8-a8a3-4754-85bb-a6ac18661119/30b02bb2-f8cb-4680-8b4d-b295fc1d5eb5"
-          (reference "R8") (unit 1)
+          (reference "R7") (unit 1)
         )
         (path "/603d0a2e-fca7-40af-8fa8-51b59d823d4d/9e308de8-a8a3-4754-85bb-a6ac18661119/94e5bb90-2559-4272-9ede-e05d2b13ade3"
-          (reference "R12") (unit 1)
+          (reference "R11") (unit 1)
         )
         (path "/603d0a2e-fca7-40af-8fa8-51b59d823d4d/9e308de8-a8a3-4754-85bb-a6ac18661119/94790e5e-8f24-4c34-8306-22332d8b1ca9"
-          (reference "R14") (unit 1)
+          (reference "R13") (unit 1)
         )
         (path "/603d0a2e-fca7-40af-8fa8-51b59d823d4d/9e308de8-a8a3-4754-85bb-a6ac18661119/74392b1e-46e8-4b44-bc27-ba912a8cb60e"
-          (reference "R16") (unit 1)
+          (reference "R15") (unit 1)
         )
         (path "/603d0a2e-fca7-40af-8fa8-51b59d823d4d/9e308de8-a8a3-4754-85bb-a6ac18661119/a5b6bf10-8ef8-4d7b-b15a-e29c9cdfd37d"
-          (reference "R18") (unit 1)
+          (reference "R17") (unit 1)
         )
       )
@@
   (symbol (lib_id "PC12311NSZ1B:PC12311NSZ1B") (at 147.32 101.6 0) (unit 1)
     (in_bom yes) (on_board yes) (dnp no) (fields_autoplaced)
-    (property "Reference" "U1" (at 146.05 85.09 0)
+    (property "Reference" "U8" (at 146.05 85.09 0)
       (effects (font (size 1.27 1.27)))
     )
@@
       (project "Addressable_Coolant_Controller"
         (path "/603d0a2e-fca7-40af-8fa8-51b59d823d4d/9e308de8-a8a3-4754-85bb-a6ac18661119/e62a760e-c259-4531-98bc-86b90a2bedbf"
+          (reference "U8") (unit 1)
+        )
+        (path "/603d0a2e-fca7-40af-8fa8-51b59d823d4d/9e308de8-a8a3-4754-85bb-a6ac18661119/67f15ca6-662b-4b8a-b540-a2e48d49f414"
+          (reference "U6") (unit 1)
+        )
+        (path "/603d0a2e-fca7-40af-8fa8-51b59d823d4d/9e308de8-a8a3-4754-85bb-a6ac18661119/ed455ca9-960e-4436-b117-323138e12946"
+          (reference "U4") (unit 1)
+        )
+        (path "/603d0a2e-fca7-40af-8fa8-51b59d823d4d/9e308de8-a8a3-4754-85bb-a6ac18661119/30b02bb2-f8cb-4680-8b4d-b295fc1d5eb5"
+          (reference "U3") (unit 1)
+        )
+        (path "/603d0a2e-fca7-40af-8fa8-51b59d823d4d/9e308de8-a8a3-4754-85bb-a6ac18661119/94e5bb90-2559-4272-9ede-e05d2b13ade3"
+          (reference "U2") (unit 1)
+        )
+        (path "/603d0a2e-fca7-40af-8fa8-51b59d823d4d/9e308de8-a8a3-4754-85bb-a6ac18661119/94790e5e-8f24-4c34-8306-22332d8b1ca9"
           (reference "U1") (unit 1)
         )
-        (path "/603d0a2e-fca7-40af-8fa8-51b59d823d4d/9e308de8-a8a3-4754-85bb-a6ac18661119/67f15ca6-662b-4b8a-b540-a2e48d49f414"
-          (reference "U2") (unit 1)
-        )
-        (path "/603d0a2e-fca7-40af-8fa8-51b59d823d4d/9e308de8-a8a3-4754-85bb-a6ac18661119/ed455ca9-960e-4436-b117-323138e12946"
-          (reference "U3") (unit 1)
-        )
-        (path "/603d0a2e-fca7-40af-8fa8-51b59d823d4d/9e308de8-a8a3-4754-85bb-a6ac18661119/30b02bb2-f8cb-4680-8b4d-b295fc1d5eb5"
-          (reference "U4") (unit 1)
-        )
-        (path "/603d0a2e-fca7-40af-8fa8-51b59d823d4d/9e308de8-a8a3-4754-85bb-a6ac18661119/94e5bb90-2559-4272-9ede-e05d2b13ade3"
-          (reference "U6") (unit 1)
-        )
-        (path "/603d0a2e-fca7-40af-8fa8-51b59d823d4d/9e308de8-a8a3-4754-85bb-a6ac18661119/94790e5e-8f24-4c34-8306-22332d8b1ca9"
-          (reference "U7") (unit 1)
-        )
         (path "/603d0a2e-fca7-40af-8fa8-51b59d823d4d/9e308de8-a8a3-4754-85bb-a6ac18661119/74392b1e-46e8-4b44-bc27-ba912a8cb60e"
-          (reference "U8") (unit 1)
+          (reference "U5") (unit 1)
         )
         (path "/603d0a2e-fca7-40af-8fa8-51b59d823d4d/9e308de8-a8a3-4754-85bb-a6ac18661119/a5b6bf10-8ef8-4d7b-b15a-e29c9cdfd37d"
-          (reference "U9") (unit 1)
+          (reference "U7") (unit 1)
         )
       )
@@
   (symbol (lib_id "Device:R") (at 125.73 92.71 90) (unit 1)
     (in_bom yes) (on_board yes) (dnp no) (fields_autoplaced)
-    (property "Reference" "R1" (at 125.73 86.36 90)
+    (property "Reference" "R2" (at 125.73 86.36 90)
       (effects (font (size 1.27 1.27)))
     )
@@
       (project "Addressable_Coolant_Controller"
         (path "/603d0a2e-fca7-40af-8fa8-51b59d823d4d/9e308de8-a8a3-4754-85bb-a6ac18661119/e62a760e-c259-4531-98bc-86b90a2bedbf"
-          (reference "R1") (unit 1)
+          (reference "R2") (unit 1)
         )
         (path "/603d0a2e-fca7-40af-8fa8-51b59d823d4d/9e308de8-a8a3-4754-85bb-a6ac18661119/67f15ca6-662b-4b8a-b540-a2e48d49f414"
-          (reference "R3") (unit 1)
+          (reference "R4") (unit 1)
         )
         (path "/603d0a2e-fca7-40af-8fa8-51b59d823d4d/9e308de8-a8a3-4754-85bb-a6ac18661119/ed455ca9-960e-4436-b117-323138e12946"
-          (reference "R5") (unit 1)
+          (reference "R6") (unit 1)
         )
         (path "/603d0a2e-fca7-40af-8fa8-51b59d823d4d/9e308de8-a8a3-4754-85bb-a6ac18661119/30b02bb2-f8cb-4680-8b4d-b295fc1d5eb5"
-          (reference "R7") (unit 1)
+          (reference "R8") (unit 1)
         )
         (path "/603d0a2e-fca7-40af-8fa8-51b59d823d4d/9e308de8-a8a3-4754-85bb-a6ac18661119/94e5bb90-2559-4272-9ede-e05d2b13ade3"
-          (reference "R11") (unit 1)
+          (reference "R12") (unit 1)
         )
         (path "/603d0a2e-fca7-40af-8fa8-51b59d823d4d/9e308de8-a8a3-4754-85bb-a6ac18661119/94790e5e-8f24-4c34-8306-22332d8b1ca9"
-          (reference "R13") (unit 1)
+          (reference "R14") (unit 1)
         )
         (path "/603d0a2e-fca7-40af-8fa8-51b59d823d4d/9e308de8-a8a3-4754-85bb-a6ac18661119/74392b1e-46e8-4b44-bc27-ba912a8cb60e"
-          (reference "R15") (unit 1)
+          (reference "R16") (unit 1)
         )
         (path "/603d0a2e-fca7-40af-8fa8-51b59d823d4d/9e308de8-a8a3-4754-85bb-a6ac18661119/a5b6bf10-8ef8-4d7b-b15a-e29c9cdfd37d"
-          (reference "R17") (unit 1)
+          (reference "R18") (unit 1)
         )
       )

Commit message: Routed connector PCB and fixed components designators
Parts:
- renumbered D1 to D8, K1 to K8, LED1 to LED8, R1 to R8, R2 to R88

Commit message: Updating Cree LED footprints with STEP files
Parts:
- LED8: footprint CreeLED Blue:C503B_BCN_CV0Z0461 -> C503B_BCN_CV0Z0461:C503B_BCN_CV0Z0461
Changed lines of the file:
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@@
       (effects (font (size 1.524 1.524)) (justify right))
     )
-    (property "Footprint" "CreeLED Blue:C503B_BCN_CV0Z0461" (at 162.56 66.04 0)
+    (property "Footprint" "C503B_BCN_CV0Z0461:C503B_BCN_CV0Z0461" (at 162.56 66.04 0)
       (effects (font (size 1.27 1.27) italic) hide)
     )
